Commit message: Add articulated Panda gripper support to ZitiBot mmp_panda.
This ports the starter-style finger joints and gripper task control so the mobile manipulator has a proper hand model with stable impedance-based finger behavior.

Made-with: Cursor

File: urdf_models/mmp_panda/mmp_panda.urdf (robot description, URDF)
Before this commit: robot mmp_panda, 11 links, 10 joints
Links:
- added link leftfinger, mass 0.1; collision box size=0.02 0.01 0.02; visual mesh filename=../panda/meshes/visual/finger.obj
- added link rightfinger, mass 0.1; collision box size=0.02 0.01 0.02; visual mesh filename=../panda/meshes/visual/finger.obj
- link link7: geometry visual mesh filename=../panda/meshes/visual/hand.obj; visual mesh filename=../panda/meshes/visual/link7.obj
Joints:
- added joint finger_joint1: type prismatic, parent link7, child leftfinger, origin xyz=0 0 0.1654 rpy=0 0 -0.78539816339, axis 0 1 0, limit lower=0.0 upper=0.04 effort=20 velocity=0.2
- added joint finger_joint2: type prismatic, parent link7, child rightfinger, origin xyz=0 0 0.1654 rpy=0 0 -0.78539816339, axis 0 1 0, limit lower=-0.04 upper=0 effort=20 velocity=0.2
