Commit message: Grasp and pour: FSM, Redis bowl goals, base to pour pose, wrist tilt
Controller state machine with hover, grasp dwells, lift, joint-hold base
move to pour target, then pour tilt about world Y. Simviz EE goal Redis
keys and debug print. World scene updates; remove cup placeholder box
visual; EmptyBowl mesh assets. Panda URDF gripper/collision tweaks for
grasp experiments.

Co-authored-by: Cursor <cursoragent@cursor.com>

File: urdf_models/mmp_panda/mmp_panda.urdf (robot description, URDF)
Before this commit: robot mmp_panda, 13 links, 12 joints
Links:
- link base_link: geometry collision box size=1.0 1.0 0.36; visual mesh filename=meshes/panda_BaseCombo.obj
- link leftfinger: geometry visual mesh filename=../panda/meshes/visual/finger.obj
- link link1: geometry collision mesh filename=../panda/meshes/collision/link1.obj; visual mesh filename=../panda/meshes/visual/link1.obj
- link link2: geometry collision mesh filename=../panda/meshes/collision/link2.obj; visual mesh filename=../panda/meshes/visual/link2.obj
- link link3: geometry collision mesh filename=../panda/meshes/collision/link3.obj; visual mesh filename=../panda/meshes/visual/link3.obj
- link link4: geometry collision mesh filename=../panda/meshes/collision/link4.obj; visual mesh filename=../panda/meshes/visual/link4.obj
- link link5: geometry collision mesh filename=../panda/meshes/collision/link5.obj; visual mesh filename=../panda/meshes/visual/link5.obj
- link link6: geometry collision mesh filename=../panda/meshes/collision/link6.obj; visual mesh filename=../panda/meshes/visual/link6.obj
- link rightfinger: geometry visual mesh filename=../panda/meshes/visual/finger.obj
